File: UFF_Stroboscope/UFF_Stroboscope.kicad_sch (KiCad schematic)
At the start: 24 parts

Commit message: v0.2 Arduino Nano was added
Parts:
- added A?: Arduino_Nano_v3.x, Module:Arduino_Nano, symbol MCU_Module:Arduino_Nano_v3.x
Changed lines of the file:
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@@
     (pin "1")
+  )
+  (symbol (lib_id "MCU_Module:Arduino_Nano_v3.x") (at 144.78 124.46 0) (unit 1)
+    (in_bom yes) (on_board yes) (fields_autoplaced)
+    (property "Reference" "A?" (id 0) (at 149.3394 149.86 0)
+      (effects (font (size 1.27 1.27)) (justify left))
+    )
+    (property "Value" "Arduino_Nano_v3.x" (id 1) (at 149.3394 152.4 0)
+      (effects (font (size 1.27 1.27)) (justify left))
+    )
+    (property "Footprint" "Module:Arduino_Nano" (id 2) (at 144.78 124.46 0)
+      (effects (font (size 1.27 1.27) italic) hide)
+    )
+    (property "Datasheet" "http://www.mouser.com/pdfdocs/Gravitech_Arduino_Nano3_0.pdf" (id 3) (at 144.78 124.46 0)
+      (effects (font (size 1.27 1.27)) hide)
+    )
+    (pin "1")
+    (pin "10")
+    (pin "11")
+    (pin "12")
+    (pin "13")
+    (pin "14")
+    (pin "15")
+    (pin "16")
+    (pin "17")
+    (pin "18")
+    (pin "19")
+    (pin "2")
+    (pin "20")
+    (pin "21")
+    (pin "22")
+    (pin "23")
+    (pin "24")
+    (pin "25")
+    (pin "26")
+    (pin "27")
+    (pin "28")
+    (pin "29")
+    (pin "3")
+    (pin "30")
+    (pin "4")
+    (pin "5")
+    (pin "6")
+    (pin "7")
+    (pin "8")
+    (pin "9")
   )
   (symbol (lib_id "Device:LED") (at 218.44 81.28 180) (unit 1)
@@
       (reference "#PWR?") (unit 1) (value "Earth") (footprint "")
     )
+    (path "/27b4db04-f796-4c7e-b32b-8e2d78ab1a23"
+      (reference "A?") (unit 1) (value "Arduino_Nano_v3.x") (footprint "Module:Arduino_Nano")
+    )
     (path "/0cb94767-4c91-43c0-9c31-4589da6c8e47"
